File: amr_audio_card/amr_audio_card.kicad_sch (KiCad schematic)
At the start: 1 part

Commit message: generate gerbers
Parts:
- added J1: Conn_Coaxial, Connector_Coaxial:BNC_TEConnectivity_1478035_Horizontal, symbol Connector:Conn_Coaxial
- added J2: USB_A, Connector_USB:USB_A_Molex_67643_Horizontal, symbol Connector:USB_A
- U1: renamed from U?; footprint (none) -> Bus-Connector:BUS_AMR
Connections:
- net GND: now also U1.A12 (GND), U1.A14 (GND), J1.2 (Ext), J2.4 (GND), J2.5 (Shield)
- net at U1.A10 (USB+): now also J2.3 (D+)
- net at U1.A11 (USB-): now also J2.2 (D-)
- net at U1.A13 (S/P-DIF_IN): now also J1.1 (In)
- net at U1.A7 (+5Vdual/+5VSB): now also J2.1 (VBUS)

Commit message: add an actual RCA jack
Parts:
- J1: footprint Connector_Coaxial:BNC_TEConnectivity_1478035_Horizontal -> Bus-Connector:Cinch
Changed lines of the file:
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@@
       (effects (font (size 1.27 1.27)) (justify left))
     )
-    (property "Footprint" "Connector_Coaxial:BNC_TEConnectivity_1478035_Horizontal" (id 2) (at 193.04 107.95 0)
+    (property "Footprint" "Bus-Connector:Cinch" (id 2) (at 193.04 107.95 0)
       (effects (font (size 1.27 1.27)) hide)
     )
@@
     )
     (path "/04ec7212-ba44-4b77-9c0d-01871e3f58e7"
-      (reference "J1") (unit 1) (value "Conn_Coaxial") (footprint "Connector_Coaxial:BNC_TEConnectivity_1478035_Horizontal")
+      (reference "J1") (unit 1) (value "Conn_Coaxial") (footprint "Bus-Connector:Cinch")
     )
     (path "/6a906923-f937-40cd-af23-ae8aab63e958"
